Commit message: 机械臂+小车模型小车可以移动

File: probot_description/urdf/PROBOT_Husky/husky.urdf.xacro (robot description, xacro)
@@ -27,4 +27,5 @@
   <xacro:include filename="$(find probot_description)/urdf/PROBOT_Husky/accessories/sick_lms1xx_mount.urdf.xacro"/>
   <xacro:include filename="$(find probot_description)/urdf/PROBOT_Husky/accessories/sensor_arch.urdf.xacro"/>
+  <xacro:include filename="$(find probot_description)/urdf/PROBOT_C800/macro_probot_c8001.xacro" />
   <property name="M_PI" value="3.14159"/>
   <!-- Base Size -->
@@ -105,4 +106,10 @@
     </xacro:husky_wheel>
     <xacro:husky_decorate />
+    <xacro:arm_probot_c8001/>
+      <joint name="c800_arm_base" type="fixed">
+        <parent link="top_plate_link" />
+        <child link="c800_base_link" />
+        <origin xyz="-0.05 0 0.02" rpy="0.0 0.0 -1.57" />
+      </joint>
       <sick_lms1xx_mount prefix="base" topic="scan"/>
       <joint name="laser_mount_joint" type="fixed">

Commit message: 添加moveit功能包和键盘控制节点

File: probot_description/urdf/PROBOT_Husky/husky.urdf.xacro (robot description, xacro)
@@ -110,5 +110,5 @@
         <parent link="top_plate_link" />
         <child link="c800_base_link" />
-        <origin xyz="-0.05 0 0.02" rpy="0.0 0.0 -1.57" />
+        <origin xyz="-0.05 0 0.12" rpy="0.0 0.0 -1.57" />
       </joint>
       <sick_lms1xx_mount prefix="base" topic="scan"/>
