Commit message: 添加运动控制demo

File: probot_description/urdf/PROBOT_C800/macro_probot_c8002.xacro (robot description, xacro)
@@ -7,5 +7,5 @@
   <xacro:arm_probot_c8001/>
   <xacro:robotiq_85_gripper prefix="" parent="link_6" >
-    <origin xyz="0.01 0 0" rpy="0 0 0"/>
+    <origin xyz="0.05 0 0" rpy="0 0 0"/>
   </xacro:robotiq_85_gripper>
  </xacro:macro>
