Commit message: 甲爪可以抓取了

File: probot_description/urdf/PROBOT_C800/macro_probot_c8001.xacro (robot description, xacro)
@@ -270,6 +270,6 @@
       xyz="0 0 1" />
     <limit
-      lower="-3"
-      upper="3"
+      lower="-1.5"
+      upper="1.5"
       effort="100"
       velocity="3" />

File: probot_description/urdf/PROBOT_C800/macro_probot_c8002.xacro (robot description, xacro)
@@ -6,6 +6,7 @@
   <xacro:include filename="$(find pr2_description)/urdf/common.xacro" />
   <xacro:arm_probot_c8001/>
+555
   <xacro:robotiq_85_gripper prefix="" parent="link_6" >
-    <origin xyz="0.05 0 0" rpy="0 0 0"/>
+    <origin xyz="0.01 0 0" rpy="0 0 0"/>
   </xacro:robotiq_85_gripper>
  </xacro:macro>

File: robotiq_85_gripper/robotiq_85_description/urdf/robotiq_85_gripper.urdf.xacro (robot description, xacro)
@@ -308,4 +308,9 @@
               <palm_link>link_6</palm_link>
               <gripper_link>gripper_finger1_finger_tip_link</gripper_link>
+              <gripper_link>gripper_finger2_finger_tip_link</gripper_link>
+              <gripper_link>gripper_finger1_inner_knuckle_link</gripper_link>
+              <gripper_link>gripper_finger2_inner_knuckle_link</gripper_link>
+              <gripper_link>gripper_finger1_knuckle_link</gripper_link>
+              <gripper_link>gripper_finger2_knuckle_link</gripper_link>
               <gripper_link>link_6</gripper_link>
             </arm>
