Commit message: 优化代码

File: probot_description/urdf/PROBOT_C800/macro_probot_c800Arm.xacro (robot description, xacro)
@@ -1,9 +1,8 @@
 <?xml version="1.0" encoding="utf-8"?>
 <robot name="probot_c800"  xmlns:xacro="http://ros.org/wiki/xacro">
+  <xacro:macro name="arm_probot_c800Arm">
   <xacro:property name="M_PI" value="3.1415926536"/>
-  <xacro:include filename="$(find probot_description)/urdf/PROBOT_C800/sensors/d435.urdf.xacro" />
-  <xacro:include filename="$(find probot_description)/urdf/PROBOT_C800/sensors/realsense.gazebo.xacro"/>
-  <link
-    name="base_link">
+  <link
+    name="c800_base_link">
     <inertial>
       <origin
@@ -11,5 +10,5 @@
         rpy="0 0 0" />
       <mass
-        value="0.468" />
+        value="4" />
       <inertia
         ixx="0.00059509"
@@ -51,5 +50,5 @@
         rpy="0 0 0" />
       <mass
-        value="1.88922089243828" />
+        value="1.7" />
       <inertia
         ixx="0.00408865798627214"
@@ -91,5 +90,5 @@
       rpy="${M_PI} 0 ${-M_PI/2}" />
     <parent
-      link="base_link" />
+      link="c800_base_link" />
     <child
       link="link_1" />
@@ -109,5 +108,5 @@
         rpy="0 0 0" />
       <mass
-        value="5.06786745806782" />
+        value="1.3" />
       <inertia
         ixx="0.0121779083694365"
@@ -167,5 +166,5 @@
         rpy="0 0 0" />
       <mass
-        value="2.47377025000813" />
+        value="1.2" />
       <inertia
         ixx="0.00663956391078891"
@@ -225,5 +224,5 @@
         rpy="0 0 0" />
       <mass
-        value="0.695111684391091" />
+        value="1.2" />
       <inertia
         ixx="0.000790631110631163"
@@ -271,6 +270,6 @@
       xyz="0 0 1" />
     <limit
-      lower="-3"
-      upper="3"
+      lower="-1.5"
+      upper="1.5"
       effort="100"
       velocity="3" />
@@ -283,5 +282,5 @@
         rpy="0 0 0" />
       <mass
-        value="0.690365366275584" />
+        value="1.2" />
       <inertia
         ixx="0.000621780696658123"
@@ -341,5 +340,5 @@
         rpy="0 0 0" />
       <mass
-        value="0.138913647701422" />
+        value="0.188913647701422" />
       <inertia
         ixx="0.000114113868764739"
@@ -398,7 +397,4 @@
     <child link="tool0" />
   </joint>
-  <sensor_d435 parent="tool0">
-    <origin xyz="0 0 0.05" rpy="0 0 ${-M_PI/2}"/>
-  </sensor_d435>
   <!-- Transmissions for ROS Control -->
   <xacro:macro name="transmission_block" params="joint_name">
@@ -421,5 +417,5 @@
   <xacro:transmission_block joint_name="joint_6"/>
   <!-- ros_control plugin -->
-  <gazebo>
+  <!--<gazebo>
     <plugin name="gazebo_ros_control" filename="libgazebo_ros_control.so">
       <robotNamespace>/</robotNamespace>
@@ -427,4 +423,5 @@
       <legacyModeNS>true</legacyModeNS>
     </plugin>
-  </gazebo>
+  </gazebo>-->
+  </xacro:macro>
 </robot>

File: probot_description/urdf/PROBOT_C800/macro_probot_c800_with_gripper.xacro (robot description, xacro)
@@ -1,9 +1,9 @@
 <?xml version="1.0"?>
 <robot xmlns:xacro="http://www.ros.org/wiki/xacro" name="probot_c800">
- <xacro:macro name="arm_probot_c8002">
-  <xacro:include filename="$(find probot_description)/urdf/PROBOT_C800/macro_probot_c8001.xacro" />
+ <xacro:macro name="arm_probot_c800_with_gripper">
+  <xacro:include filename="$(find probot_description)/urdf/PROBOT_C800/macro_probot_c800Arm.xacro" />
   <xacro:include filename="$(find robotiq_85_description)/urdf/robotiq_85_gripper.urdf.xacro" />
   <xacro:include filename="$(find pr2_description)/urdf/common.xacro" />
-  <xacro:arm_probot_c8001/>
+  <xacro:arm_probot_c800Arm/>
 555
   <xacro:robotiq_85_gripper prefix="" parent="link_6" >

File: probot_description/urdf/PROBOT_HuskyArm/huskyArm.urdf.xacro (robot description, xacro)
@@ -27,5 +27,5 @@
   <xacro:include filename="$(find probot_description)/urdf/PROBOT_HuskyArm/accessories/sick_lms1xx_mount.urdf.xacro"/>
   <xacro:include filename="$(find probot_description)/urdf/PROBOT_HuskyArm/accessories/sensor_arch.urdf.xacro"/>
-  <xacro:include filename="$(find probot_description)/urdf/PROBOT_C800/macro_probot_c8002.xacro" />
+  <xacro:include filename="$(find probot_description)/urdf/PROBOT_C800/macro_probot_c800_with_gripper.xacro" />
   <property name="M_PI" value="3.14159"/>
   <!-- Base Size -->
@@ -107,5 +107,5 @@
     </xacro:husky_wheel>
     <xacro:husky_decorate />
-    <xacro:arm_probot_c8002/>
+    <xacro:arm_probot_c800_with_gripper/>
       <joint name="c800_arm_base" type="fixed">
         <parent link="top_plate_link" />
