Commit message: 备份

File: probot_description/urdf/PROBOT_HuskyArm/huskyArm.urdf.xacro (robot description, xacro)
@@ -48,4 +48,5 @@
           <mesh filename="package://probot_description/meshes/PROBOT_Husky/base_link.dae" />
         </geometry>
+        <material name="orange" />
       </visual>
       <collision>

File: robotiq_85_gripper/robotiq_85_description/urdf/robotiq_85_gripper.urdf.xacro (robot description, xacro)
@@ -20,5 +20,5 @@
             </collision>
             <inertial>
-                <mass value="0.636951" />
+                <mass value="0.0006951" />
                 <origin xyz="0.0 0.0 0.0" />
                 <inertia ixx = "0.000380" ixy = "0.000000" ixz = "0.000000"
@@ -61,5 +61,5 @@
             </collision>
             <inertial>
-                <mass value="0.018491" />
+                <mass value="0.0008491" />
                 <origin xyz="0.0 0.0 0.0" />
                 <inertia ixx = "0.000009" ixy = "-0.000001" ixz = "0.000000"
@@ -69,4 +69,5 @@
         </link>
         <gazebo reference="${prefix}gripper_finger1_knuckle_link">
+            <material>Gazebo/Blue</material>
             <implicitSpringDamper>1</implicitSpringDamper>
             <mu1>100000</mu1>
@@ -87,5 +88,5 @@
             </collision>
             <inertial>
-                <mass value="0.018491" />
+                <mass value="0.000218491" />
                 <origin xyz="0.0 0.0 0.0" />
                 <inertia ixx = "0.000009" ixy = "-0.000001" ixz = "0.000000"
@@ -123,5 +124,5 @@
             </collision>
             <inertial>
-                <mass value="0.027309" />
+                <mass value="0.000227309" />
                 <origin xyz="0.0 0.0 0.0" />
                 <inertia ixx = "0.000003" ixy = "-0.000002" ixz = "0.000000"
@@ -131,4 +132,5 @@
         </link>
         <gazebo reference="${prefix}gripper_finger1_finger_link">
+            <material>Gazebo/Blue</material>
             <implicitSpringDamper>1</implicitSpringDamper>
             <mu1>100000</mu1>
@@ -149,5 +151,5 @@
             </collision>
             <inertial>
-                <mass value="0.027309" />
+                <mass value="0.000227309" />
                 <origin xyz="0.0 0.0 0.0" />
                 <inertia ixx = "0.000003" ixy = "-0.000002" ixz = "0.000000"
@@ -157,4 +159,5 @@
         </link>
         <gazebo reference="${prefix}gripper_finger2_finger_link">
+            <material>Gazebo/Blue</material>
             <implicitSpringDamper>1</implicitSpringDamper>
             <mu1>100000</mu1>
@@ -191,5 +194,5 @@
             </collision>
             <inertial>
-                <mass value="0.029951" />
+                <mass value="0.000229951" />
                 <origin xyz="0.0 0.0 0.0" />
                 <inertia ixx = "0.000039" ixy = "0.000000" ixz = "0.000000"
@@ -217,5 +220,5 @@
             </collision>
             <inertial>
-                <mass value="0.029951" />
+                <mass value="0.000229951" />
                 <origin xyz="0.0 0.0 0.0" />
                 <inertia ixx = "0.000039" ixy = "0.000000" ixz = "0.000000"
@@ -259,5 +262,5 @@
             </collision>
             <inertial>
-                <mass value="0.019555" />
+                <mass value="0.000219555" />
                 <origin xyz="0.0 0.0 0.0" />
                 <inertia ixx = "0.000002" ixy = "0.000000" ixz = "0.000000"
@@ -285,5 +288,5 @@
             </collision>
             <inertial>
-                <mass value="0.019555" />
+                <mass value="0.00019555" />
                 <origin xyz="0.0 0.0 0.0" />
                 <inertia ixx = "0.000002" ixy = "0.000000" ixz = "0.000000"
